Commit message: added more links

File: urdf/my3darm.xacro (robot description, xacro)
@@ -71,3 +71,35 @@
       </visual>
   </link>
+  <joint name="link_03__link_04" type="revolute">
+    <axis xyz="0 1 0"/>
+    <limit effort="1000.0" lower="-3.14" upper="3.14" velocity="0.5"/>
+    <origin rpy="0 0 0" xyz="-1.287 0 0.057"/>
+    <parent link="link_03"/>
+    <child link="link_04"/>
+  </joint>
+  <link name="link_04">
+      <visual>
+        <origin rpy="0 0 0" xyz="-0.05 0 0" />
+        <geometry>
+          <mesh filename="package://mrm2/meshes/Link4_reduced.stl" scale="0.01 0.01 0.01" />
+        </geometry>
+        <material name="orange" />
+      </visual>
+  </link>
+  <joint name="link_04__link_05" type="revolute">
+    <axis xyz="0 1 0"/>
+    <limit effort="1000.0" lower="-3.14" upper="3.14" velocity="0.5"/>
+    <origin rpy="0 0 0" xyz="-0.4327 0 0"/>
+    <parent link="link_04"/>
+    <child link="link_05"/>
+  </joint>
+  <link name="link_05">
+      <visual>
+        <origin rpy="0 0 0" xyz="0 0.0416 -0.0004" />
+        <geometry>
+          <mesh filename="package://mrm2/meshes/Link5_reduced.stl" scale="0.01 0.01 0.01" />
+        </geometry>
+        <material name="red" />
+      </visual>
+  </link>
 </robot>

Commit message: Added Link5

File: urdf/my3darm.xacro (robot description, xacro)
@@ -88,5 +88,5 @@
   </link>
   <joint name="link_04__link_05" type="revolute">
-    <axis xyz="0 1 0"/>
+    <axis xyz="1 0 0"/>
     <limit effort="1000.0" lower="-3.14" upper="3.14" velocity="0.5"/>
     <origin rpy="0 0 0" xyz="-0.4327 0 0"/>
@@ -96,5 +96,5 @@
   <link name="link_05">
       <visual>
-        <origin rpy="0 0 0" xyz="0 0.0416 -0.0004" />
+        <origin rpy="0 0 0" xyz="0 0.0005 0.0416" />
         <geometry>
           <mesh filename="package://mrm2/meshes/Link5_reduced.stl" scale="0.01 0.01 0.01" />

Commit message: Added grippers

File: urdf/my3darm.xacro (robot description, xacro)
@@ -8,5 +8,5 @@
   </material>
   <material name="malachita">
-    <color rgba="64 0 230 1" />
+    <color rgba="64 0 230 0.25" />
   </material>
   <material name="electric_indigo">
@@ -103,3 +103,35 @@
       </visual>
   </link>
+  <joint name="link_05__gripper_01" type="revolute">
+    <axis xyz="0 0 1"/>
+    <limit effort="1000.0" lower="-3.14" upper="3.14" velocity="0.5"/>
+    <origin rpy="0 0 0" xyz="0 -0.1225 -0.1605"/>
+    <parent link="link_05"/>
+    <child link="gripper_01"/>
+  </joint>
+  <link name="gripper_01">
+      <visual>
+        <origin rpy="0 0 0" xyz="-0.19 -0.04 0" />
+        <geometry>
+          <mesh filename="package://mrm2/meshes/Gripper1_reduced.stl" scale="0.01 0.01 0.01" />
+        </geometry>
+        <material name="malachita" />
+      </visual>
+  </link>
+  <joint name="link_05__gripper_02" type="revolute">
+    <axis xyz="0 0 1"/>
+    <limit effort="1000.0" lower="-3.14" upper="3.14" velocity="0.5"/>
+    <origin rpy="0 0 0" xyz="0 0.1225 -0.1605"/>
+    <parent link="link_05"/>
+    <child link="gripper_02"/>
+  </joint>
+  <link name="gripper_02">
+      <visual>
+        <origin rpy="0 0 0" xyz="-0.19 0.039 0" />
+        <geometry>
+          <mesh filename="package://mrm2/meshes/Gripper2_reduced.stl" scale="0.01 0.01 0.01" />
+        </geometry>
+        <material name="electric_indigo" />
+      </visual>
+  </link>
 </robot>

Commit message: Link5.stl corrected

File: urdf/my3darm.xacro (robot description, xacro)
@@ -8,5 +8,5 @@
   </material>
   <material name="malachita">
-    <color rgba="64 0 230 0.25" />
+    <color rgba="64 0 230 1" />
   </material>
   <material name="electric_indigo">
@@ -18,5 +18,4 @@
         <geometry>
           <mesh filename="package://mrm2/meshes/Base_reduced.stl" scale="0.01 0.01 0.01" />
-          <!-- <box size="1.623 0.6400 0.4500" /> -->
         </geometry>
         <material name="orange" />

Commit message: Added collision tags

File: urdf/my3darm.xacro (robot description, xacro)
@@ -1,4 +1,4 @@
 <?xml version="1.0" ?>
-<robot name="popo" xmlns:xacro="http://www.ros.org/wiki/xacro">
+<robot name="my3darm" xmlns:xacro="http://www.ros.org/wiki/xacro">
   <material name="orange">
     <color rgba="84 211 0 1" />
@@ -21,4 +21,10 @@
         <material name="orange" />
       </visual>
+      <collision>
+        <origin rpy="0 0 0" xyz="0 0 0.225" />
+        <geometry>
+          <mesh filename="package://mrm2/meshes/Base_reduced.stl" scale ="0.001 0.001 0.001"/>
+        </geometry>
+      </collision>
   </link>
   <joint name="base_link__link_01" type="revolute">
@@ -30,11 +36,17 @@
   </joint>
   <link name="link_01">
-      <visual>
-        <origin rpy="0 0 0" xyz="0 0 0.1875" />
-        <geometry>
-          <mesh filename="package://mrm2/meshes/Link1_reduced.stl" scale="0.01 0.01 0.01" />
-        </geometry>
-        <material name="red" />
-      </visual>
+    <visual>
+      <origin rpy="0 0 0" xyz="0 0 0.1875" />
+      <geometry>
+        <mesh filename="package://mrm2/meshes/Link1_reduced.stl" scale="0.01 0.01 0.01" />
+      </geometry>
+      <material name="red" />
+    </visual>
+    <collision>
+      <origin rpy="0 0 0" xyz="0 0 0.1875" />
+      <geometry>
+        <mesh filename="package://mrm2/meshes/Link1_reduced.stl" scale="0.01 0.01 0.01" />
+      </geometry>
+    </collision>
   </link>
   <joint name="link_01__link_02" type="revolute">
@@ -46,11 +58,17 @@
   </joint>
   <link name="link_02">
-      <visual>
-        <origin rpy="0 0 0" xyz="0 0 0.58323" />
-        <geometry>
-          <mesh filename="package://mrm2/meshes/Link2_reduced.stl" scale="0.01 0.01 0.01" />
-        </geometry>
-        <material name="malachita" />
-      </visual>
+    <visual>
+      <origin rpy="0 0 0" xyz="0 0 0.58323" />
+      <geometry>
+        <mesh filename="package://mrm2/meshes/Link2_reduced.stl" scale="0.01 0.01 0.01" />
+      </geometry>
+      <material name="malachita" />
+    </visual>
+    <collision>
+      <origin rpy="0 0 0" xyz="0 0 0.58323" />
+      <geometry>
+        <mesh filename="package://mrm2/meshes/Link2_reduced.stl" scale="0.01 0.01 0.01" />
+      </geometry>
+    </collision>
   </link>
   <joint name="link_02__link_03" type="revolute">
@@ -62,11 +80,17 @@
   </joint>
   <link name="link_03">
-      <visual>
-        <origin rpy="0 0 0" xyz="-0.65 0 0" />
-        <geometry>
-          <mesh filename="package://mrm2/meshes/Link3_reduced.stl" scale="0.01 0.01 0.01" />
-        </geometry>
-        <material name="electric_indigo" />
-      </visual>
+    <visual>
+      <origin rpy="0 0 0" xyz="-0.65 0 0" />
+      <geometry>
+        <mesh filename="package://mrm2/meshes/Link3_reduced.stl" scale="0.01 0.01 0.01" />
+      </geometry>
+      <material name="electric_indigo" />
+    </visual>
+    <collision>
+      <origin rpy="0 0 0" xyz="-0.65 0 0" />
+      <geometry>
+        <mesh filename="package://mrm2/meshes/Link3_reduced.stl" scale="0.01 0.01 0.01" />
+      </geometry>
+    </collision>
   </link>
   <joint name="link_03__link_04" type="revolute">
@@ -78,11 +102,17 @@
   </joint>
   <link name="link_04">
-      <visual>
-        <origin rpy="0 0 0" xyz="-0.05 0 0" />
-        <geometry>
-          <mesh filename="package://mrm2/meshes/Link4_reduced.stl" scale="0.01 0.01 0.01" />
-        </geometry>
-        <material name="orange" />
-      </visual>
+    <visual>
+      <origin rpy="0 0 0" xyz="-0.05 0 0" />
+      <geometry>
+        <mesh filename="package://mrm2/meshes/Link4_reduced.stl" scale="0.01 0.01 0.01" />
+      </geometry>
+      <material name="orange" />
+    </visual>
+    <collision>
+      <origin rpy="0 0 0" xyz="-0.05 0 0" />
+      <geometry>
+        <mesh filename="package://mrm2/meshes/Link4_reduced.stl" scale="0.01 0.01 0.01" />
+      </geometry>
+    </collision>
   </link>
   <joint name="link_04__link_05" type="revolute">
@@ -94,11 +124,17 @@
   </joint>
   <link name="link_05">
-      <visual>
-        <origin rpy="0 0 0" xyz="0 0.0005 0.0416" />
-        <geometry>
-          <mesh filename="package://mrm2/meshes/Link5_reduced.stl" scale="0.01 0.01 0.01" />
-        </geometry>
-        <material name="red" />
-      </visual>
+    <visual>
+      <origin rpy="0 0 0" xyz="0 0.0005 0.0416" />
+      <geometry>
+        <mesh filename="package://mrm2/meshes/Link5_reduced.stl" scale="0.01 0.01 0.01" />
+      </geometry>
+      <material name="red" />
+    </visual>
+    <collision>
+      <origin rpy="0 0 0" xyz="0 0.0005 0.0416" />
+      <geometry>
+        <mesh filename="package://mrm2/meshes/Link5_reduced.stl" scale="0.01 0.01 0.01" />
+      </geometry>
+    </collision>
   </link>
   <joint name="link_05__gripper_01" type="revolute">
@@ -110,11 +146,17 @@
   </joint>
   <link name="gripper_01">
-      <visual>
-        <origin rpy="0 0 0" xyz="-0.19 -0.04 0" />
-        <geometry>
-          <mesh filename="package://mrm2/meshes/Gripper1_reduced.stl" scale="0.01 0.01 0.01" />
-        </geometry>
-        <material name="malachita" />
-      </visual>
+    <visual>
+      <origin rpy="0 0 0" xyz="-0.19 -0.04 0" />
+      <geometry>
+        <mesh filename="package://mrm2/meshes/Gripper1_reduced.stl" scale="0.01 0.01 0.01" />
+      </geometry>
+      <material name="malachita" />
+    </visual>
+    <collision>
+      <origin rpy="0 0 0" xyz="-0.19 -0.04 0" />
+      <geometry>
+        <mesh filename="package://mrm2/meshes/Gripper1_reduced.stl" scale="0.01 0.01 0.01" />
+      </geometry>
+    </collision>
   </link>
   <joint name="link_05__gripper_02" type="revolute">
@@ -126,11 +168,17 @@
   </joint>
   <link name="gripper_02">
-      <visual>
-        <origin rpy="0 0 0" xyz="-0.19 0.039 0" />
-        <geometry>
-          <mesh filename="package://mrm2/meshes/Gripper2_reduced.stl" scale="0.01 0.01 0.01" />
-        </geometry>
-        <material name="electric_indigo" />
-      </visual>
+    <visual>
+      <origin rpy="0 0 0" xyz="-0.19 0.039 0" />
+      <geometry>
+        <mesh filename="package://mrm2/meshes/Gripper2_reduced.stl" scale="0.01 0.01 0.01" />
+      </geometry>
+      <material name="electric_indigo" />
+    </visual>
+    <collision>
+      <origin rpy="0 0 0" xyz="-0.19 0.039 0" />
+      <geometry>
+        <mesh filename="package://mrm2/meshes/Gripper2_reduced.stl" scale="0.01 0.01 0.01" />
+      </geometry>
+    </collision>
   </link>
 </robot>

Commit message: renaming according to the convetion used by the guys at https://rds.theconstructsim.com/

File: urdf/my3darm.xacro (robot description, xacro)
@@ -17,5 +17,5 @@
         <origin rpy="0 0 0" xyz="0 0 0.225" />
         <geometry>
-          <mesh filename="package://mrm2/meshes/Base_reduced.stl" scale="0.01 0.01 0.01" />
+          <mesh filename="package://my3dbotarm_description/meshes/Base_reduced.stl" scale="0.01 0.01 0.01" />
         </geometry>
         <material name="orange" />
@@ -24,5 +24,5 @@
         <origin rpy="0 0 0" xyz="0 0 0.225" />
         <geometry>
-          <mesh filename="package://mrm2/meshes/Base_reduced.stl" scale ="0.001 0.001 0.001"/>
+          <mesh filename="package://my3dbotarm_description/meshes/Base_reduced.stl" scale ="0.001 0.001 0.001"/>
         </geometry>
       </collision>
@@ -39,5 +39,5 @@
       <origin rpy="0 0 0" xyz="0 0 0.1875" />
       <geometry>
-        <mesh filename="package://mrm2/meshes/Link1_reduced.stl" scale="0.01 0.01 0.01" />
+        <mesh filename="package://my3dbotarm_description/meshes/Link1_reduced.stl" scale="0.01 0.01 0.01" />
       </geometry>
       <material name="red" />
@@ -46,5 +46,5 @@
       <origin rpy="0 0 0" xyz="0 0 0.1875" />
       <geometry>
-        <mesh filename="package://mrm2/meshes/Link1_reduced.stl" scale="0.01 0.01 0.01" />
+        <mesh filename="package://my3dbotarm_description/meshes/Link1_reduced.stl" scale="0.01 0.01 0.01" />
       </geometry>
     </collision>
@@ -61,5 +61,5 @@
       <origin rpy="0 0 0" xyz="0 0 0.58323" />
       <geometry>
-        <mesh filename="package://mrm2/meshes/Link2_reduced.stl" scale="0.01 0.01 0.01" />
+        <mesh filename="package://my3dbotarm_description/meshes/Link2_reduced.stl" scale="0.01 0.01 0.01" />
       </geometry>
       <material name="malachita" />
@@ -68,5 +68,5 @@
       <origin rpy="0 0 0" xyz="0 0 0.58323" />
       <geometry>
-        <mesh filename="package://mrm2/meshes/Link2_reduced.stl" scale="0.01 0.01 0.01" />
+        <mesh filename="package://my3dbotarm_description/meshes/Link2_reduced.stl" scale="0.01 0.01 0.01" />
       </geometry>
     </collision>
@@ -83,5 +83,5 @@
       <origin rpy="0 0 0" xyz="-0.65 0 0" />
       <geometry>
-        <mesh filename="package://mrm2/meshes/Link3_reduced.stl" scale="0.01 0.01 0.01" />
+        <mesh filename="package://my3dbotarm_description/meshes/Link3_reduced.stl" scale="0.01 0.01 0.01" />
       </geometry>
       <material name="electric_indigo" />
@@ -90,5 +90,5 @@
       <origin rpy="0 0 0" xyz="-0.65 0 0" />
       <geometry>
-        <mesh filename="package://mrm2/meshes/Link3_reduced.stl" scale="0.01 0.01 0.01" />
+        <mesh filename="package://my3dbotarm_description/meshes/Link3_reduced.stl" scale="0.01 0.01 0.01" />
       </geometry>
     </collision>
@@ -105,5 +105,5 @@
       <origin rpy="0 0 0" xyz="-0.05 0 0" />
       <geometry>
-        <mesh filename="package://mrm2/meshes/Link4_reduced.stl" scale="0.01 0.01 0.01" />
+        <mesh filename="package://my3dbotarm_description/meshes/Link4_reduced.stl" scale="0.01 0.01 0.01" />
       </geometry>
       <material name="orange" />
@@ -112,5 +112,5 @@
       <origin rpy="0 0 0" xyz="-0.05 0 0" />
       <geometry>
-        <mesh filename="package://mrm2/meshes/Link4_reduced.stl" scale="0.01 0.01 0.01" />
+        <mesh filename="package://my3dbotarm_description/meshes/Link4_reduced.stl" scale="0.01 0.01 0.01" />
       </geometry>
     </collision>
@@ -127,5 +127,5 @@
       <origin rpy="0 0 0" xyz="0 0.0005 0.0416" />
       <geometry>
-        <mesh filename="package://mrm2/meshes/Link5_reduced.stl" scale="0.01 0.01 0.01" />
+        <mesh filename="package://my3dbotarm_description/meshes/Link5_reduced.stl" scale="0.01 0.01 0.01" />
       </geometry>
       <material name="red" />
@@ -134,5 +134,5 @@
       <origin rpy="0 0 0" xyz="0 0.0005 0.0416" />
       <geometry>
-        <mesh filename="package://mrm2/meshes/Link5_reduced.stl" scale="0.01 0.01 0.01" />
+        <mesh filename="package://my3dbotarm_description/meshes/Link5_reduced.stl" scale="0.01 0.01 0.01" />
       </geometry>
     </collision>
@@ -149,5 +149,5 @@
       <origin rpy="0 0 0" xyz="-0.19 -0.04 0" />
       <geometry>
-        <mesh filename="package://mrm2/meshes/Gripper1_reduced.stl" scale="0.01 0.01 0.01" />
+        <mesh filename="package://my3dbotarm_description/meshes/Gripper1_reduced.stl" scale="0.01 0.01 0.01" />
       </geometry>
       <material name="malachita" />
@@ -156,5 +156,5 @@
       <origin rpy="0 0 0" xyz="-0.19 -0.04 0" />
       <geometry>
-        <mesh filename="package://mrm2/meshes/Gripper1_reduced.stl" scale="0.01 0.01 0.01" />
+        <mesh filename="package://my3dbotarm_description/meshes/Gripper1_reduced.stl" scale="0.01 0.01 0.01" />
       </geometry>
     </collision>
@@ -171,5 +171,5 @@
       <origin rpy="0 0 0" xyz="-0.19 0.039 0" />
       <geometry>
-        <mesh filename="package://mrm2/meshes/Gripper2_reduced.stl" scale="0.01 0.01 0.01" />
+        <mesh filename="package://my3dbotarm_description/meshes/Gripper2_reduced.stl" scale="0.01 0.01 0.01" />
       </geometry>
       <material name="electric_indigo" />
@@ -178,5 +178,5 @@
       <origin rpy="0 0 0" xyz="-0.19 0.039 0" />
       <geometry>
-        <mesh filename="package://mrm2/meshes/Gripper2_reduced.stl" scale="0.01 0.01 0.01" />
+        <mesh filename="package://my3dbotarm_description/meshes/Gripper2_reduced.stl" scale="0.01 0.01 0.01" />
       </geometry>
     </collision>

Commit message: commenting material tags for links because they render ugly on rviz

File: urdf/my3darm.xacro (robot description, xacro)
@@ -5,5 +5,5 @@
   </material>
   <material name="red">
-    <color rgba="77 5 232 1" />
+    <color rgba="207 0 15 1" />
   </material>
   <material name="malachita">
@@ -19,5 +19,5 @@
           <mesh filename="package://my3dbotarm_description/meshes/Base_reduced.stl" scale="0.01 0.01 0.01" />
         </geometry>
-        <material name="orange" />
+	<!-- <material name="orange" /> -->
       </visual>
       <collision>
@@ -41,5 +41,5 @@
         <mesh filename="package://my3dbotarm_description/meshes/Link1_reduced.stl" scale="0.01 0.01 0.01" />
       </geometry>
-      <material name="red" />
+      <!-- <material name="red" /> -->
     </visual>
     <collision>
@@ -63,5 +63,5 @@
         <mesh filename="package://my3dbotarm_description/meshes/Link2_reduced.stl" scale="0.01 0.01 0.01" />
       </geometry>
-      <material name="malachita" />
+      <!-- <material name="malachita" /> -->
     </visual>
     <collision>
@@ -85,5 +85,5 @@
         <mesh filename="package://my3dbotarm_description/meshes/Link3_reduced.stl" scale="0.01 0.01 0.01" />
       </geometry>
-      <material name="electric_indigo" />
+      <!-- <material name="electric_indigo" /> -->
     </visual>
     <collision>
@@ -107,5 +107,5 @@
         <mesh filename="package://my3dbotarm_description/meshes/Link4_reduced.stl" scale="0.01 0.01 0.01" />
       </geometry>
-      <material name="orange" />
+      <!-- <material name="orange" /> -->
     </visual>
     <collision>
@@ -129,5 +129,5 @@
         <mesh filename="package://my3dbotarm_description/meshes/Link5_reduced.stl" scale="0.01 0.01 0.01" />
       </geometry>
-      <material name="red" />
+      <!-- <material name="red" /> -->
     </visual>
     <collision>
@@ -151,5 +151,5 @@
         <mesh filename="package://my3dbotarm_description/meshes/Gripper1_reduced.stl" scale="0.01 0.01 0.01" />
       </geometry>
-      <material name="malachita" />
+      <!-- <material name="malachita" /> -->
     </visual>
     <collision>
@@ -173,5 +173,5 @@
         <mesh filename="package://my3dbotarm_description/meshes/Gripper2_reduced.stl" scale="0.01 0.01 0.01" />
       </geometry>
-      <material name="electric_indigo" />
+      <!-- <material name="electric_indigo" /> -->
     </visual>
     <collision>
