Commit message: changed the urdf scale to mm

File: urdf/my3darm.xacro (robot description, xacro)
@@ -15,12 +15,12 @@
   <link name="base_link">
       <visual>
-        <origin rpy="0 0 0" xyz="0 0 0.225" />
+        <origin rpy="0 0 0" xyz="0 0 0.0225" />
         <geometry>
-          <mesh filename="package://my3dbotarm_description/meshes/Base_reduced.stl" scale="0.01 0.01 0.01" />
+          <mesh filename="package://my3dbotarm_description/meshes/Base_reduced.stl" scale="0.001 0.001 0.001" />
         </geometry>
-	<!-- <material name="orange" /> -->
+	<material name="orange" />
       </visual>
       <collision>
-        <origin rpy="0 0 0" xyz="0 0 0.225" />
+        <origin rpy="0 0 0" xyz="0 0 0.0225" />
         <geometry>
           <mesh filename="package://my3dbotarm_description/meshes/Base_reduced.stl" scale ="0.001 0.001 0.001"/>
@@ -31,5 +31,5 @@
     <axis xyz="0 0 1"/>
     <limit effort="1000.0" lower="-3.14" upper="3.14" velocity="0.5"/>
-    <origin rpy="0 0 0" xyz="-0.386 0 0.425"/>
+    <origin rpy="0 0 0" xyz="-0.0386 0 0.0425"/>
     <parent link="base_link"/>
     <child link="link_01"/>
@@ -37,14 +37,14 @@
   <link name="link_01">
     <visual>
-      <origin rpy="0 0 0" xyz="0 0 0.1875" />
+      <origin rpy="0 0 0" xyz="0 0 0.01875" />
       <geometry>
-        <mesh filename="package://my3dbotarm_description/meshes/Link1_reduced.stl" scale="0.01 0.01 0.01" />
+        <mesh filename="package://my3dbotarm_description/meshes/Link1_reduced.stl" scale="0.001 0.001 0.001" />
       </geometry>
-      <!-- <material name="red" /> -->
+      <material name="red" />
     </visual>
     <collision>
-      <origin rpy="0 0 0" xyz="0 0 0.1875" />
+      <origin rpy="0 0 0" xyz="0 0 0.01875" />
       <geometry>
-        <mesh filename="package://my3dbotarm_description/meshes/Link1_reduced.stl" scale="0.01 0.01 0.01" />
+        <mesh filename="package://my3dbotarm_description/meshes/Link1_reduced.stl" scale="0.001 0.001 0.001" />
       </geometry>
     </collision>
@@ -53,5 +53,5 @@
     <axis xyz="0 1 0"/>
     <limit effort="1000.0" lower="-3.14" upper="3.14" velocity="0.5"/>
-    <origin rpy="0 0 0" xyz="0 0 0.2500431"/>
+    <origin rpy="0 0 0" xyz="0 0 0.02500431"/>
     <parent link="link_01"/>
     <child link="link_02"/>
@@ -59,14 +59,14 @@
   <link name="link_02">
     <visual>
-      <origin rpy="0 0 0" xyz="0 0 0.58323" />
+      <origin rpy="0 0 0" xyz="0 0 0.058323" />
       <geometry>
-        <mesh filename="package://my3dbotarm_description/meshes/Link2_reduced.stl" scale="0.01 0.01 0.01" />
+        <mesh filename="package://my3dbotarm_description/meshes/Link2_reduced.stl" scale="0.001 0.001 0.001" />
       </geometry>
-      <!-- <material name="malachita" /> -->
+      <material name="malachita" />
     </visual>
     <collision>
-      <origin rpy="0 0 0" xyz="0 0 0.58323" />
+      <origin rpy="0 0 0" xyz="0 0 0.058323" />
       <geometry>
-        <mesh filename="package://my3dbotarm_description/meshes/Link2_reduced.stl" scale="0.01 0.01 0.01" />
+        <mesh filename="package://my3dbotarm_description/meshes/Link2_reduced.stl" scale="0.001 0.001 0.001" />
       </geometry>
     </collision>
@@ -75,5 +75,5 @@
     <axis xyz="0 1 0"/>
     <limit effort="1000.0" lower="-3.14" upper="3.14" velocity="0.5"/>
-    <origin rpy="0 0 0" xyz="0 0 1.073"/>
+    <origin rpy="0 0 0" xyz="0 0 0.1073"/>
     <parent link="link_02"/>
     <child link="link_03"/>
@@ -81,14 +81,14 @@
   <link name="link_03">
     <visual>
-      <origin rpy="0 0 0" xyz="-0.65 0 0" />
+      <origin rpy="0 0 0" xyz="-0.065 0 0" />
       <geometry>
-        <mesh filename="package://my3dbotarm_description/meshes/Link3_reduced.stl" scale="0.01 0.01 0.01" />
+        <mesh filename="package://my3dbotarm_description/meshes/Link3_reduced.stl" scale="0.001 0.001 0.001" />
       </geometry>
-      <!-- <material name="electric_indigo" /> -->
+      <material name="electric_indigo" />
     </visual>
     <collision>
-      <origin rpy="0 0 0" xyz="-0.65 0 0" />
+      <origin rpy="0 0 0" xyz="-0.065 0 0" />
       <geometry>
-        <mesh filename="package://my3dbotarm_description/meshes/Link3_reduced.stl" scale="0.01 0.01 0.01" />
+        <mesh filename="package://my3dbotarm_description/meshes/Link3_reduced.stl" scale="0.001 0.001 0.001" />
       </geometry>
     </collision>
@@ -97,5 +97,5 @@
     <axis xyz="0 1 0"/>
     <limit effort="1000.0" lower="-3.14" upper="3.14" velocity="0.5"/>
-    <origin rpy="0 0 0" xyz="-1.287 0 0.057"/>
+    <origin rpy="0 0 0" xyz="-0.1287 0 0.0057"/>
     <parent link="link_03"/>
     <child link="link_04"/>
@@ -103,14 +103,14 @@
   <link name="link_04">
     <visual>
-      <origin rpy="0 0 0" xyz="-0.05 0 0" />
+      <origin rpy="0 0 0" xyz="-0.005 0 0" />
       <geometry>
-        <mesh filename="package://my3dbotarm_description/meshes/Link4_reduced.stl" scale="0.01 0.01 0.01" />
+        <mesh filename="package://my3dbotarm_description/meshes/Link4_reduced.stl" scale="0.001 0.001 0.001" />
       </geometry>
-      <!-- <material name="orange" /> -->
+      <material name="orange" />
     </visual>
     <collision>
-      <origin rpy="0 0 0" xyz="-0.05 0 0" />
+      <origin rpy="0 0 0" xyz="-0.005 0 0" />
       <geometry>
-        <mesh filename="package://my3dbotarm_description/meshes/Link4_reduced.stl" scale="0.01 0.01 0.01" />
+        <mesh filename="package://my3dbotarm_description/meshes/Link4_reduced.stl" scale="0.001 0.001 0.001" />
       </geometry>
     </collision>
@@ -119,5 +119,5 @@
     <axis xyz="1 0 0"/>
     <limit effort="1000.0" lower="-3.14" upper="3.14" velocity="0.5"/>
-    <origin rpy="0 0 0" xyz="-0.4327 0 0"/>
+    <origin rpy="0 0 0" xyz="-0.04327 0 0"/>
     <parent link="link_04"/>
     <child link="link_05"/>
@@ -125,14 +125,14 @@
   <link name="link_05">
     <visual>
-      <origin rpy="0 0 0" xyz="0 0.0005 0.0416" />
+      <origin rpy="0 0 0" xyz="0 0.00005 0.00416" />
       <geometry>
-        <mesh filename="package://my3dbotarm_description/meshes/Link5_reduced.stl" scale="0.01 0.01 0.01" />
+        <mesh filename="package://my3dbotarm_description/meshes/Link5_reduced.stl" scale="0.001 0.001 0.001" />
       </geometry>
-      <!-- <material name="red" /> -->
+      <material name="red" />
     </visual>
     <collision>
-      <origin rpy="0 0 0" xyz="0 0.0005 0.0416" />
+      <origin rpy="0 0 0" xyz="0 0.00005 0.00416" />
       <geometry>
-        <mesh filename="package://my3dbotarm_description/meshes/Link5_reduced.stl" scale="0.01 0.01 0.01" />
+        <mesh filename="package://my3dbotarm_description/meshes/Link5_reduced.stl" scale="0.001 0.001 0.001" />
       </geometry>
     </collision>
@@ -141,5 +141,5 @@
     <axis xyz="0 0 1"/>
     <limit effort="1000.0" lower="-3.14" upper="3.14" velocity="0.5"/>
-    <origin rpy="0 0 0" xyz="0 -0.1225 -0.1605"/>
+    <origin rpy="0 0 0" xyz="0 -0.01225 -0.01605"/>
     <parent link="link_05"/>
     <child link="gripper_01"/>
@@ -147,14 +147,14 @@
   <link name="gripper_01">
     <visual>
-      <origin rpy="0 0 0" xyz="-0.19 -0.04 0" />
+      <origin rpy="0 0 0" xyz="-0.019 -0.004 0" />
       <geometry>
-        <mesh filename="package://my3dbotarm_description/meshes/Gripper1_reduced.stl" scale="0.01 0.01 0.01" />
+        <mesh filename="package://my3dbotarm_description/meshes/Gripper1_reduced.stl" scale="0.001 0.001 0.001" />
       </geometry>
-      <!-- <material name="malachita" /> -->
+      <material name="malachita" />
     </visual>
     <collision>
-      <origin rpy="0 0 0" xyz="-0.19 -0.04 0" />
+      <origin rpy="0 0 0" xyz="-0.019 -0.004 0" />
       <geometry>
-        <mesh filename="package://my3dbotarm_description/meshes/Gripper1_reduced.stl" scale="0.01 0.01 0.01" />
+        <mesh filename="package://my3dbotarm_description/meshes/Gripper1_reduced.stl" scale="0.001 0.001 0.001" />
       </geometry>
     </collision>
@@ -163,5 +163,5 @@
     <axis xyz="0 0 1"/>
     <limit effort="1000.0" lower="-3.14" upper="3.14" velocity="0.5"/>
-    <origin rpy="0 0 0" xyz="0 0.1225 -0.1605"/>
+    <origin rpy="0 0 0" xyz="0 0.01225 -0.01605"/>
     <parent link="link_05"/>
     <child link="gripper_02"/>
@@ -169,14 +169,14 @@
   <link name="gripper_02">
     <visual>
-      <origin rpy="0 0 0" xyz="-0.19 0.039 0" />
+      <origin rpy="0 0 0" xyz="-0.019 0.0039 0" />
       <geometry>
-        <mesh filename="package://my3dbotarm_description/meshes/Gripper2_reduced.stl" scale="0.01 0.01 0.01" />
+        <mesh filename="package://my3dbotarm_description/meshes/Gripper2_reduced.stl" scale="0.001 0.001 0.001" />
       </geometry>
-      <!-- <material name="electric_indigo" /> -->
+      <material name="electric_indigo" />
     </visual>
     <collision>
-      <origin rpy="0 0 0" xyz="-0.19 0.039 0" />
+      <origin rpy="0 0 0" xyz="-0.019 0.0039 0" />
       <geometry>
-        <mesh filename="package://my3dbotarm_description/meshes/Gripper2_reduced.stl" scale="0.01 0.01 0.01" />
+        <mesh filename="package://my3dbotarm_description/meshes/Gripper2_reduced.stl" scale="0.001 0.001 0.001" />
       </geometry>
     </collision>

Commit message: adjust lower and upper values more accuratetly

File: urdf/my3darm.xacro (robot description, xacro)
@@ -19,5 +19,5 @@
           <mesh filename="package://my3dbotarm_description/meshes/Base_reduced.stl" scale="0.001 0.001 0.001" />
         </geometry>
-	<material name="orange" />
+	      <material name="orange" />
       </visual>
       <collision>
@@ -30,5 +30,5 @@
   <joint name="base_link__link_01" type="revolute">
     <axis xyz="0 0 1"/>
-    <limit effort="1000.0" lower="-3.14" upper="3.14" velocity="0.5"/>
+    <limit effort="1000.0" lower="-1.5" upper="1.5" velocity="0.5"/>
     <origin rpy="0 0 0" xyz="-0.0386 0 0.0425"/>
     <parent link="base_link"/>
@@ -52,5 +52,5 @@
   <joint name="link_01__link_02" type="revolute">
     <axis xyz="0 1 0"/>
-    <limit effort="1000.0" lower="-3.14" upper="3.14" velocity="0.5"/>
+    <limit effort="1000.0" lower="-1.5" upper="1.5" velocity="0.5"/>
     <origin rpy="0 0 0" xyz="0 0 0.02500431"/>
     <parent link="link_01"/>
@@ -74,5 +74,5 @@
   <joint name="link_02__link_03" type="revolute">
     <axis xyz="0 1 0"/>
-    <limit effort="1000.0" lower="-3.14" upper="3.14" velocity="0.5"/>
+    <limit effort="1000.0" lower="-1.5" upper="1.5" velocity="0.5"/>
     <origin rpy="0 0 0" xyz="0 0 0.1073"/>
     <parent link="link_02"/>
@@ -96,5 +96,5 @@
   <joint name="link_03__link_04" type="revolute">
     <axis xyz="0 1 0"/>
-    <limit effort="1000.0" lower="-3.14" upper="3.14" velocity="0.5"/>
+    <limit effort="1000.0" lower="-1.5" upper="1.5" velocity="0.5"/>
     <origin rpy="0 0 0" xyz="-0.1287 0 0.0057"/>
     <parent link="link_03"/>
@@ -118,5 +118,5 @@
   <joint name="link_04__link_05" type="revolute">
     <axis xyz="1 0 0"/>
-    <limit effort="1000.0" lower="-3.14" upper="3.14" velocity="0.5"/>
+    <limit effort="1000.0" lower="-1.5" upper="1.5" velocity="0.5"/>
     <origin rpy="0 0 0" xyz="-0.04327 0 0"/>
     <parent link="link_04"/>
@@ -140,5 +140,5 @@
   <joint name="link_05__gripper_01" type="revolute">
     <axis xyz="0 0 1"/>
-    <limit effort="1000.0" lower="-3.14" upper="3.14" velocity="0.5"/>
+    <limit effort="1000.0" lower="-1.5" upper="1.5" velocity="0.5"/>
     <origin rpy="0 0 0" xyz="0 -0.01225 -0.01605"/>
     <parent link="link_05"/>
@@ -162,5 +162,5 @@
   <joint name="link_05__gripper_02" type="revolute">
     <axis xyz="0 0 1"/>
-    <limit effort="1000.0" lower="-3.14" upper="3.14" velocity="0.5"/>
+    <limit effort="1000.0" lower="-1.5" upper="1.5" velocity="0.5"/>
     <origin rpy="0 0 0" xyz="0 0.01225 -0.01605"/>
     <parent link="link_05"/>
