Commit message: Last adjustments to generate ikfast plugin correctly... I guess...

File: urdf/my3dbotarm.xacro (robot description, xacro)
@@ -1,4 +1,4 @@
 <?xml version="1.0" ?>
-<robot name="my3darm" xmlns:xacro="http://www.ros.org/wiki/xacro">
+<robot name="my3dbotarm" xmlns:xacro="http://www.ros.org/wiki/xacro">
   <material name="orange">
     <color rgba="84 211 0 1" />
@@ -13,5 +13,5 @@
     <color rgba="140 252 20 1" />
   </material>
-  <link name="base_link">
+  <link name="base">
       <visual>
         <origin rpy="0 0 0" xyz="0 0 0.0225" />
@@ -28,9 +28,9 @@
       </collision>
   </link>
-  <joint name="base_link__link_01" type="revolute">
+  <joint name="base__link_01" type="revolute">
     <axis xyz="0 0 1"/>
     <limit effort="1000.0" lower="-1.5" upper="1.5" velocity="0.5"/>
     <origin rpy="0 0 0" xyz="-0.0386 0 0.0425"/>
-    <parent link="base_link"/>
+    <parent link="base"/>
     <child link="link_01"/>
   </joint>

Commit message: velocity changed to 1.0

File: urdf/my3dbotarm.xacro (robot description, xacro)
@@ -30,5 +30,5 @@
   <joint name="base__link_01" type="revolute">
     <axis xyz="0 0 1"/>
-    <limit effort="1000.0" lower="-1.5" upper="1.5" velocity="0.5"/>
+    <limit effort="1000.0" lower="-1.5" upper="1.5" velocity="1.0"/>
     <origin rpy="0 0 0" xyz="-0.0386 0 0.0425"/>
     <parent link="base"/>
@@ -52,5 +52,5 @@
   <joint name="link_01__link_02" type="revolute">
     <axis xyz="0 1 0"/>
-    <limit effort="1000.0" lower="-1.5" upper="1.5" velocity="0.5"/>
+    <limit effort="1000.0" lower="-1.5" upper="1.5" velocity="1.0"/>
     <origin rpy="0 0 0" xyz="0 0 0.02500431"/>
     <parent link="link_01"/>
@@ -74,5 +74,5 @@
   <joint name="link_02__link_03" type="revolute">
     <axis xyz="0 1 0"/>
-    <limit effort="1000.0" lower="-1.5" upper="1.5" velocity="0.5"/>
+    <limit effort="1000.0" lower="-1.5" upper="1.5" velocity="1.0"/>
     <origin rpy="0 0 0" xyz="0 0 0.1073"/>
     <parent link="link_02"/>
@@ -96,5 +96,5 @@
   <joint name="link_03__link_04" type="revolute">
     <axis xyz="0 1 0"/>
-    <limit effort="1000.0" lower="-1.5" upper="1.5" velocity="0.5"/>
+    <limit effort="1000.0" lower="-1.5" upper="1.5" velocity="1.0"/>
     <origin rpy="0 0 0" xyz="-0.1287 0 0.0057"/>
     <parent link="link_03"/>
@@ -118,5 +118,5 @@
   <joint name="link_04__link_05" type="revolute">
     <axis xyz="1 0 0"/>
-    <limit effort="1000.0" lower="-1.5" upper="1.5" velocity="0.5"/>
+    <limit effort="1000.0" lower="-1.5" upper="1.5" velocity="1.0"/>
     <origin rpy="0 0 0" xyz="-0.04327 0 0"/>
     <parent link="link_04"/>
@@ -140,5 +140,5 @@
   <joint name="link_05__gripper_01" type="revolute">
     <axis xyz="0 0 1"/>
-    <limit effort="1000.0" lower="-1.5" upper="1.5" velocity="0.5"/>
+    <limit effort="1000.0" lower="-1.5" upper="1.5" velocity="1.0"/>
     <origin rpy="0 0 0" xyz="0 -0.01225 -0.01605"/>
     <parent link="link_05"/>
@@ -162,5 +162,5 @@
   <joint name="link_05__gripper_02" type="revolute">
     <axis xyz="0 0 1"/>
-    <limit effort="1000.0" lower="-1.5" upper="1.5" velocity="0.5"/>
+    <limit effort="1000.0" lower="-1.5" upper="1.5" velocity="1.0"/>
     <origin rpy="0 0 0" xyz="0 0.01225 -0.01605"/>
     <parent link="link_05"/>
